Commit message: add gazebo model for zed2 stereo

File: zed_wrapper/urdf/zed_descr.urdf.xacro (robot description, xacro)
@@ -16,4 +16,5 @@
 -->
 <robot name="stereolabs_camera" xmlns:xacro="http://ros.org/wiki/xacro">
+  <xacro:arg name="robot_name"   default="zed" />
   <xacro:arg name="camera_name"   default="zed" />
   <xacro:arg name="camera_model"  default="zed" />
@@ -25,5 +26,6 @@
   <xacro:arg name="gnss_z" default="0.0" />
   <xacro:include filename="$(find zed_wrapper)/urdf/zed_macro.urdf.xacro" />
-  <xacro:zed_camera name="$(arg camera_name)" model="$(arg camera_model)" custom_baseline="$(arg custom_baseline)" enable_gnss="$(arg enable_gnss)">
+  <xacro:zed_camera robot_name="$(arg robot_name)"
+      name="$(arg camera_name)" model="$(arg camera_model)" custom_baseline="$(arg custom_baseline)" enable_gnss="$(arg enable_gnss)">
 	    <origin xyz="$(arg gnss_x) $(arg gnss_y) $(arg gnss_z)" rpy="0 0 0"/>
   </xacro:zed_camera>

File: zed_wrapper/urdf/zed_macro.urdf.xacro (robot description, xacro)
@@ -17,4 +17,5 @@
 <robot xmlns:xacro="http://wiki.ros.org/xacro">
   <xacro:include filename="$(find zed_wrapper)/urdf/include/materials.urdf.xacro" />
+  <xacro:include filename="$(find zed_wrapper)/gazebo/zed.gazebo.xacro" />
   <xacro:property name="M_PI"     value="3.1415926535897931" />
   <!--
@@ -24,5 +25,5 @@
       - enable_gnss: if true enable the URDF link
   -->
-  <xacro:macro name="zed_camera" params="name=zed model=zed enable_gnss=false custom_baseline=0 *gnss_origin">
+  <xacro:macro name="zed_camera" params="parent robot_name:=zed name=zed model=zed enable_gnss=false custom_baseline=0 *origin gazebo:=false">
     <xacro:if value="${model == 'zed'}">
       <xacro:property name="baseline" value="0.12" />
@@ -83,4 +84,9 @@
     <!-- Camera mounting point (the threaded screw hole in the bottom) -->
     <link name="${name}_camera_link" />
+    <joint name="${name}_joint" type="fixed">
+      <xacro:insert_block name="origin" />
+      <parent link="${parent}"/>
+      <child link="${name}_camera_link" />
+    </joint>
     <!-- Camera Center -->
     <link name="${name}_camera_center">
@@ -89,5 +95,5 @@
           <origin xyz="${screw_offset_x} 0 ${screw_offset_z}" rpy="0 0 0"/>
           <geometry>
-            <mesh filename="package://zed_interfaces/meshes/${model}.stl" />
+            <mesh filename="file://$(find zed_interfaces)/meshes/${model}.stl" />
           </geometry>
           <material name="${model}_mat" />
@@ -96,5 +102,5 @@
           <origin xyz="${screw_offset_x} 0 ${screw_offset_z}" rpy="0 0 0"/>
           <geometry>
-            <mesh filename="package://zed_interfaces/meshes/${model}.stl" />
+            <mesh filename="file://$(find zed_interfaces)/meshes/${model}.stl" />
           </geometry>
         </collision>
@@ -108,9 +114,9 @@
     <!-- Left Camera -->
     <link name="${name}_left_camera_frame">
-      <xacro:if value="${model == 'virtual'}">
+      <xacro:unless value="${model == 'virtual'}">
         <visual>
           <origin xyz="0 0 0" rpy="0 0 0"/>
           <geometry>
-            <mesh filename="package://zed_interfaces/meshes/${model}.stl" />
+            <mesh filename="file://$(find zed_interfaces)/meshes/${model}.stl" />
           </geometry>
           <material name="${model}_mat" />
@@ -119,8 +125,8 @@
           <origin xyz="0 0 0" rpy="0 0 0"/>
           <geometry>
-            <mesh filename="package://zed_interfaces/meshes/${model}.stl" />
+            <mesh filename="file://$(find zed_interfaces)/meshes/${model}.stl" />
           </geometry>
         </collision>
-      </xacro:if>
+      </xacro:unless>
     </link>
     <joint name="${name}_left_camera_joint" type="fixed">
@@ -137,9 +143,9 @@
     <!-- Right Camera -->
     <link name="${name}_right_camera_frame">
-      <xacro:if value="${model == 'virtual'}">
+      <xacro:unless value="${model == 'virtual'}">
         <visual>
           <origin xyz="0 0 0" rpy="0 0 0"/>
           <geometry>
-            <mesh filename="package://zed_interfaces/meshes/${model}.stl" />
+            <mesh filename="file://$(find zed_interfaces)/meshes/${model}.stl" />
           </geometry>
           <material name="${model}_mat" />
@@ -148,8 +154,8 @@
           <origin xyz="0 0 0" rpy="0 0 0"/>
           <geometry>
-            <mesh filename="package://zed_interfaces/meshes/${model}.stl" />
+            <mesh filename="file://$(find zed_interfaces)/meshes/${model}.stl" />
           </geometry>
         </collision>
-      </xacro:if>
+      </xacro:unless>
     </link>
     <joint name="${name}_right_camera_joint" type="fixed">
@@ -196,6 +202,18 @@
         <parent link="${name}_camera_link"/>
         <child link="${name}_gnss_link"/>
-        <xacro:insert_block name="gnss_origin" />
-      </joint>
+        <xacro:insert_block name="origin" />
+      </joint>
+    </xacro:if>
+    <xacro:if value="${gazebo}">
+      <xacro:gazebo_zed
+        robot_name="${robot_name}"
+        camera_name="${name}"
+        reference_link="${name}_camera_link"
+        left_frame="${name}_left_camera_frame"
+        right_frame="${name}_right_camera_frame"
+        width="1920"
+        height="1080"
+        fps="30"
+      />
     </xacro:if>
   </xacro:macro>
