Commit message: take image width and height as parameters

File: zed_wrapper/urdf/zed_macro.urdf.xacro (robot description, xacro)
@@ -25,5 +25,5 @@
       - enable_gnss: if true enable the URDF link
   -->
-  <xacro:macro name="zed_camera" params="parent robot_name:=zed name=zed model=zed enable_gnss=false custom_baseline=0 *origin gazebo:=false">
+  <xacro:macro name="zed_camera" params="parent robot_name:=zed name=zed model=zed enable_gnss=false custom_baseline=0 *origin gazebo:=false image_width:=1920 image_height:=1080 fps:=30">
     <xacro:if value="${model == 'zed'}">
       <xacro:property name="baseline" value="0.12" />
@@ -212,7 +212,7 @@
         left_frame="${name}_left_camera_frame"
         right_frame="${name}_right_camera_frame"
-        width="1920"
-        height="1080"
-        fps="30"
+        width="${image_width}"
+        height="${image_height}"
+        fps="${fps}"
       />
     </xacro:if>

Commit message: fix wrapper for ros2 compatibility

File: zed_wrapper/urdf/zed_macro.urdf.xacro (robot description, xacro)
@@ -25,5 +25,5 @@
       - enable_gnss: if true enable the URDF link
   -->
-  <xacro:macro name="zed_camera" params="parent robot_name:=zed name=zed model=zed enable_gnss=false custom_baseline=0 *origin gazebo:=false image_width:=1920 image_height:=1080 fps:=30">
+  <xacro:macro name="zed_camera" params="parent:=base_link robot_name:=zed name=zed model=zed enable_gnss=false custom_baseline=0 *origin gazebo:=false image_width:=1920 image_height:=1080 fps:=30">
     <xacro:if value="${model == 'zed'}">
       <xacro:property name="baseline" value="0.12" />
@@ -84,9 +84,9 @@
     <!-- Camera mounting point (the threaded screw hole in the bottom) -->
     <link name="${name}_camera_link" />
-    <joint name="${name}_joint" type="fixed">
+    <!-- <joint name="${name}_joint" type="fixed">
       <xacro:insert_block name="origin" />
       <parent link="${parent}"/>
       <child link="${name}_camera_link" />
-    </joint>
+    </joint> -->
     <!-- Camera Center -->
     <link name="${name}_camera_center">
